Commit message: mechbase only

File: one/robots/end_effectors/linkerbot/o6/urdf/o6_left.urdf (robot description, URDF)
Before this commit: robot linkerhand_o6_left, 12 links, 11 joints
Links:
- link lh_hand_base_link: geometry collision mesh filename=../meshes/left_cvx/hand_base_link.stl; visual mesh filename=../meshes/left_cvx/hand_base_link.stl
- link lh_index_distal: geometry collision mesh filename=../meshes/left_cvx/index_distal.stl; visual mesh filename=../meshes/left_cvx/index_distal.stl
- link lh_index_proximal: geometry collision mesh filename=../meshes/left_cvx/index_proximal.stl; visual mesh filename=../meshes/left_cvx/index_proximal.stl
- link lh_middle_distal: geometry collision mesh filename=../meshes/left_cvx/middle_distal.stl; visual mesh filename=../meshes/left_cvx/middle_distal.stl
- link lh_middle_proximal: geometry collision mesh filename=../meshes/left_cvx/middle_proximal.stl; visual mesh filename=../meshes/left_cvx/middle_proximal.stl
- link lh_pinky_distal: geometry collision mesh filename=../meshes/left_cvx/pinky_distal.stl; visual mesh filename=../meshes/left_cvx/pinky_distal.stl
- link lh_pinky_proximal: geometry collision mesh filename=../meshes/left_cvx/pinky_proximal.stl; visual mesh filename=../meshes/left_cvx/pinky_proximal.stl
- link lh_ring_distal: geometry collision mesh filename=../meshes/left_cvx/ring_distal.stl; visual mesh filename=../meshes/left_cvx/ring_distal.stl
- link lh_ring_proximal: geometry collision mesh filename=../meshes/left_cvx/ring_proximal.stl; visual mesh filename=../meshes/left_cvx/ring_proximal.stl
- link lh_thumb_distal: geometry collision mesh filename=../meshes/left_cvx/thumb_distal.stl; visual mesh filename=../meshes/left_cvx/thumb_distal.stl
- link lh_thumb_metacarpals: geometry collision mesh filename=../meshes/left_cvx/thumb_metacarpals.stl; visual mesh filename=../meshes/left_cvx/thumb_metacarpals.stl
- link lh_thumb_metacarpals_base2: geometry collision mesh filename=../meshes/left_cvx/thumb_metacarpals_base2.stl; visual mesh filename=../meshes/left_cvx/thumb_metacarpals_base2.stl

File: one/robots/end_effectors/linkerbot/o6/urdf/o6_right.urdf (robot description, URDF)
Before this commit: robot linkerhand_o6_right, 12 links, 11 joints
Links:
- link rh_hand_base_link: geometry collision mesh filename=../meshes/right_cvx/hand_base_link.stl; visual mesh filename=../meshes/right_cvx/hand_base_link.stl
- link rh_index_distal: geometry collision mesh filename=../meshes/right_cvx/index_distal.stl; visual mesh filename=../meshes/right_cvx/index_distal.stl
- link rh_index_proximal: geometry collision mesh filename=../meshes/right_cvx/index_proximal.stl; visual mesh filename=../meshes/right_cvx/index_proximal.stl
- link rh_middle_distal: geometry collision mesh filename=../meshes/right_cvx/middle_distal.stl; visual mesh filename=../meshes/right_cvx/middle_distal.stl
- link rh_middle_proximal: geometry collision mesh filename=../meshes/right_cvx/middle_proximal.stl; visual mesh filename=../meshes/right_cvx/middle_proximal.stl
- link rh_pinky_distal: geometry collision mesh filename=../meshes/right_cvx/pinky_distal.stl; visual mesh filename=../meshes/right_cvx/pinky_distal.stl
- link rh_pinky_proximal: geometry collision mesh filename=../meshes/right_cvx/pinky_proximal.stl; visual mesh filename=../meshes/right_cvx/pinky_proximal.stl
- link rh_ring_distal: geometry collision mesh filename=../meshes/right_cvx/ring_distal.stl; visual mesh filename=../meshes/right_cvx/ring_distal.stl
- link rh_ring_proximal: geometry collision mesh filename=../meshes/right_cvx/ring_proximal.stl; visual mesh filename=../meshes/right_cvx/ring_proximal.stl
- link rh_thumb_distal: geometry collision mesh filename=../meshes/right_cvx/thumb_distal.stl; visual mesh filename=../meshes/right_cvx/thumb_distal.stl
- link rh_thumb_metacarpals: geometry collision mesh filename=../meshes/right_cvx/thumb_metacarpals.stl; visual mesh filename=../meshes/right_cvx/thumb_metacarpals.stl
- link rh_thumb_metacarpals_base2: geometry collision mesh filename=../meshes/right_cvx/thumb_metacarpals_base2.stl; visual mesh filename=../meshes/right_cvx/thumb_metacarpals_base2.stl

File: one/robots/humanoids/linx/l1/urdf/h0602.urdf (robot description, URDF)
Before this commit: robot , 21 links, 20 joints
Links:
- link base_link: geometry collision mesh filename=../meshes/base_link.stl; visual mesh filename=../meshes/base_link.stl
- link left_arm_link_1: geometry collision mesh filename=../meshes/left_arm_link_1.stl; visual mesh filename=../meshes/left_arm_link_1.stl
- link left_arm_link_2: geometry collision mesh filename=../meshes/left_arm_link_2.stl; visual mesh filename=../meshes/left_arm_link_2.stl
- link left_arm_link_3: geometry collision mesh filename=../meshes/left_arm_link_3.stl; visual mesh filename=../meshes/left_arm_link_3.stl
- link left_arm_link_4: geometry collision mesh filename=../meshes/left_arm_link_4.stl; visual mesh filename=../meshes/left_arm_link_4.stl
- link left_arm_link_5: geometry collision mesh filename=../meshes/left_arm_link_5.stl; visual mesh filename=../meshes/left_arm_link_5.stl
- link left_arm_link_6: geometry collision mesh filename=../meshes/left_arm_link_6.stl; visual mesh filename=../meshes/left_arm_link_6.stl
- link neck_link1: geometry collision mesh filename=../meshes/neck_link1.stl; visual mesh filename=../meshes/neck_link1.stl
- link neck_link2: geometry collision mesh filename=../meshes/neck_link2.stl; visual mesh filename=../meshes/neck_link2.stl
- link right_arm_link_1: geometry collision mesh filename=../meshes/right_arm_link_1.stl; visual mesh filename=../meshes/right_arm_link_1.stl
- link right_arm_link_2: geometry collision mesh filename=../meshes/right_arm_link_2.stl; visual mesh filename=../meshes/right_arm_link_2.stl
- link right_arm_link_3: geometry collision mesh filename=../meshes/right_arm_link_3.stl; visual mesh filename=../meshes/right_arm_link_3.stl
- link right_arm_link_4: geometry collision mesh filename=../meshes/right_arm_link_4.stl; visual mesh filename=../meshes/right_arm_link_4.stl
- link right_arm_link_5: geometry collision mesh filename=../meshes/right_arm_link_5.stl; visual mesh filename=../meshes/right_arm_link_5.stl
- link right_arm_link_6: geometry collision mesh filename=../meshes/right_arm_link_6.stl; visual mesh filename=../meshes/right_arm_link_6.stl
- link waist_link1: geometry collision mesh filename=../meshes/waist_link1.stl; visual mesh filename=../meshes/waist_link1.stl
- link waist_link2: geometry collision mesh filename=../meshes/waist_link2.stl; visual mesh filename=../meshes/waist_link2.stl
