Commit message: linkerbot o6

File: one/robots/humanoids/linx/l1/urdf/h0602.urdf (robot description, URDF)
Before this commit: robot , 45 links, 44 joints
Links:
- removed link lh_hand_base_link
- removed link lh_index_distal
- removed link lh_index_proximal
- removed link lh_middle_distal
- removed link lh_middle_proximal
- removed link lh_pinky_distal
- removed link lh_pinky_proximal
- removed link lh_ring_distal
- removed link lh_ring_proximal
- removed link lh_thumb_distal
- removed link lh_thumb_metacarpals
- removed link lh_thumb_metacarpals_base2
- removed link rh_hand_base_link
- removed link rh_index_distal
- removed link rh_index_proximal
- removed link rh_middle_distal
- removed link rh_middle_proximal
- removed link rh_pinky_distal
- removed link rh_pinky_proximal
- removed link rh_ring_distal
- removed link rh_ring_proximal
- removed link rh_thumb_distal
- removed link rh_thumb_metacarpals
- removed link rh_thumb_metacarpals_base2
Joints:
- removed joint left_linkerhand_mount_joint
- removed joint lh_index_dip
- removed joint lh_index_mcp_pitch
- removed joint lh_middle_dip
- removed joint lh_middle_mcp_pitch
- removed joint lh_pinky_dip
- removed joint lh_pinky_mcp_pitch
- removed joint lh_ring_dip
- removed joint lh_ring_mcp_pitch
- removed joint lh_thumb_cmc_pitch
- removed joint lh_thumb_cmc_yaw
- removed joint lh_thumb_ip
- removed joint rh_index_dip
- removed joint rh_index_mcp_pitch
- removed joint rh_middle_dip
- removed joint rh_middle_mcp_pitch
- removed joint rh_pinky_dip
- removed joint rh_pinky_mcp_pitch
- removed joint rh_ring_dip
- removed joint rh_ring_mcp_pitch
- removed joint rh_thumb_cmc_pitch
- removed joint rh_thumb_cmc_yaw
- removed joint rh_thumb_ip
- removed joint right_linkerhand_mount_joint

Commit message: l1

File: one/robots/humanoids/linx/l1/urdf/h0602.urdf (robot description, URDF)
Before this commit: robot , 21 links, 20 joints
Joints:
- joint left_arm_joint_2: origin xyz=0.00162414749273029 0.112000025930368 0.0485000000000013 rpy=-1.57079632679489 0 0 -> xyz=0 0.112000025930368 0.0485000000000013 rpy=-1.57079632679489 0 0
